File: Smersh2.brd (EAGLE design)
At the start: 98 x 49 mm, 133 parts

Commit message: Доработанные платы
Parts:
- added R10, R11, R14, R8, R9: 10k, resistor:R0603
- C15, C16, C17, C20, C22, C23, C28, C3, C31, C32, C33, C34, C35, C4, C5, C6: device resistor:C0805 -> resistor:C0603
- C38: device rcl:C0805 -> rcl:C0603
- R1: device rcl:R0805 -> rcl:R0603
- R18, R19, R20, R21, R22: device resistor:R0805 -> resistor:R0603
- R4: device resistor:R1206 -> resistor:R0603
- moved R4 5.83 mm to (67.7, 33.6)
- moved R7 1.07 mm to (9.36, 19.4)
- moved R12 1.00 mm to (70.5, 33.5)
Connections:
- new net N$1: ADS.2, R8.1
- new net N$17: ADS3.2, R10.2
- new net N$19: ADS1.2, R11.2
- new net N$20: R14.1, STM32.60
- new net N$4: ADS2.2, R9.1
- net +5V: now also R10.1, R11.1, R8.2, R9.2
- net GND: now also R14.2; no longer STM32.60
Routing:
- net GND: track 728.7 -> 750.5 mm, vias 19 -> 21
- net +5V: track 225.0 -> 239.8 mm
- net N$1: track 0.00 -> 7.53 mm, vias 0 -> 2
- net N$20: track 0.00 -> 4.00 mm, vias 0 -> 1
- net N$4: track 0.00 -> 3.40 mm
- net N$19: track 0.00 -> 2.35 mm
- net N$17: track 0.00 -> 2.26 mm
- net N$29: track 17.3 -> 15.5 mm, vias 1 -> 0
- net +3V3: track 329.1 -> 330.3 mm
- net MOTOR_3: track 34.7 -> 34.0 mm
