File: Smersh2.sch (EAGLE design)
At the start: 133 parts

Commit message: Доработанные платы
Parts:
- added R10, R11, R14, R8, R9: 10k, resistor:R-EU_R0603
- C15, C16, C17, C20, C22, C23, C28, C3, C31, C32, C33, C34, C35, C4, C5, C6: device resistor:C-EUC0805 -> resistor:C-EUC0603
- C38: device rcl:C-EUC0805 -> rcl:C-EUC0603
- R1: device rcl:R-EU_R0805 -> rcl:R-EU_R0603
- R18, R19, R20, R21, R22: device resistor:R-EU_R0805 -> resistor:R-EU_R0603
- R4: device resistor:R-EU_R1206 -> resistor:R-EU_R0603
Connections:
- new net N$1: ADS.ALERT/RDY, R8.1
- new net N$17: ADS3.ALERT/RDY, R10.2
- new net N$19: ADS1.ALERT/RDY, R11.2
- new net N$20: R14.1, STM32.BOOT0
- new net N$4: ADS2.ALERT/RDY, R9.1
- net +5V: now also R10.1, R11.1, R8.2, R9.2
- net GND: now also R14.2; no longer STM32.BOOT0
